File: example/LedRing.sch (KiCad schematic (older format))
At the start: 24 parts

Commit message: Reannotating
Parts:
- C10, C11, C12, C13, C14, C15, C16, C17, C18, C7, C8, C9: renamed from C?; footprint (none) -> Capacitors_SMD:C_0805
- U10, U11, U12, U13, U2, U3, U4, U5, U6, U7, U8, U9: renamed from U?; footprint (none) -> symwaf:ws2812b
Changed lines of the file:
@@
 $EndDescr
 $Comp
-L ws2812b U?
+L ws2812b U4
 U 1 1 5AA3D3BB
 P 5100 3150
-F 0 "U?" H 4900 3450 60  0000 C CNN
+F 0 "U4" H 4900 3450 60  0000 C CNN
 F 1 "ws2812b" H 5200 2850 60  0000 C CNN
-F 2 "" H 5100 3150 60  0001 C CNN
+F 2 "symwaf:ws2812b" H 5100 3150 60  0001 C CNN
 F 3 "" H 5100 3150 60  0001 C CNN
 	1    5100 3150
@@
 $EndComp
 $Comp
-L ws2812b U?
+L ws2812b U5
 U 1 1 5AA3D415
 P 6250 3150
-F 0 "U?" H 6050 3450 60  0000 C CNN
+F 0 "U5" H 6050 3450 60  0000 C CNN
 F 1 "ws2812b" H 6350 2850 60  0000 C CNN
-F 2 "" H 6250 3150 60  0001 C CNN
+F 2 "symwaf:ws2812b" H 6250 3150 60  0001 C CNN
 F 3 "" H 6250 3150 60  0001 C CNN
 	1    6250 3150
@@
 $EndComp
 $Comp
-L ws2812b U?
+L ws2812b U2
 U 1 1 5AA3D587
 P 2800 3150
-F 0 "U?" H 2600 3450 60  0000 C CNN
+F 0 "U2" H 2600 3450 60  0000 C CNN
 F 1 "ws2812b" H 2900 2850 60  0000 C CNN
-F 2 "" H 2800 3150 60  0001 C CNN
+F 2 "symwaf:ws2812b" H 2800 3150 60  0001 C CNN
 F 3 "" H 2800 3150 60  0001 C CNN
 	1    2800 3150
@@
 $EndComp
 $Comp
-L ws2812b U?
+L ws2812b U3
 U 1 1 5AA3D58D
 P 3950 3150
-F 0 "U?" H 3750 3450 60  0000 C CNN
+F 0 "U3" H 3750 3450 60  0000 C CNN
 F 1 "ws2812b" H 4050 2850 60  0000 C CNN
-F 2 "" H 3950 3150 60  0001 C CNN
+F 2 "symwaf:ws2812b" H 3950 3150 60  0001 C CNN
 F 3 "" H 3950 3150 60  0001 C CNN
 	1    3950 3150
@@
 VCC
 $Comp
-L ws2812b U?
+L ws2812b U8
 U 1 1 5AA3FDA1
 P 2800 4850
-F 0 "U?" H 2600 5150 60  0000 C CNN
+F 0 "U8" H 2600 5150 60  0000 C CNN
 F 1 "ws2812b" H 2900 4550 60  0000 C CNN
-F 2 "" H 2800 4850 60  0001 C CNN
+F 2 "symwaf:ws2812b" H 2800 4850 60  0001 C CNN
 F 3 "" H 2800 4850 60  0001 C CNN
 	1    2800 4850
@@
 $EndComp
 $Comp
-L ws2812b U?
+L ws2812b U9
 U 1 1 5AA3FDA7
 P 3950 4850
-F 0 "U?" H 3750 5150 60  0000 C CNN
+F 0 "U9" H 3750 5150 60  0000 C CNN
 F 1 "ws2812b" H 4050 4550 60  0000 C CNN
-F 2 "" H 3950 4850 60  0001 C CNN
+F 2 "symwaf:ws2812b" H 3950 4850 60  0001 C CNN
 F 3 "" H 3950 4850 60  0001 C CNN
 	1    3950 4850
@@
 $EndComp
 $Comp
-L ws2812b U?
+L ws2812b U6
 U 1 1 5AA3FDAD
 P 7400 3150
-F 0 "U?" H 7200 3450 60  0000 C CNN
+F 0 "U6" H 7200 3450 60  0000 C CNN
 F 1 "ws2812b" H 7500 2850 60  0000 C CNN
-F 2 "" H 7400 3150 60  0001 C CNN
+F 2 "symwaf:ws2812b" H 7400 3150 60  0001 C CNN
 F 3 "" H 7400 3150 60  0001 C CNN
 	1    7400 3150
@@
 $EndComp
 $Comp
-L ws2812b U?
+L ws2812b U7
 U 1 1 5AA3FDB3
 P 8550 3150
-F 0 "U?" H 8350 3450 60  0000 C CNN
+F 0 "U7" H 8350 3450 60  0000 C CNN
 F 1 "ws2812b" H 8650 2850 60  0000 C CNN
-F 2 "" H 8550 3150 60  0001 C CNN
+F 2 "symwaf:ws2812b" H 8550 3150 60  0001 C CNN
 F 3 "" H 8550 3150 60  0001 C CNN
 	1    8550 3150
@@
 $EndComp
 $Comp
-L ws2812b U?
+L ws2812b U10
 U 1 1 5AA4006D
 P 5100 4850
-F 0 "U?" H 4900 5150 60  0000 C CNN
+F 0 "U10" H 4900 5150 60  0000 C CNN
 F 1 "ws2812b" H 5200 4550 60  0000 C CNN
-F 2 "" H 5100 4850 60  0001 C CNN
+F 2 "symwaf:ws2812b" H 5100 4850 60  0001 C CNN
 F 3 "" H 5100 4850 60  0001 C CNN
 	1    5100 4850
@@
 $EndComp
 $Comp
-L ws2812b U?
+L ws2812b U11
 U 1 1 5AA40073
 P 6250 4850
-F 0 "U?" H 6050 5150 60  0000 C CNN
+F 0 "U11" H 6050 5150 60  0000 C CNN
 F 1 "ws2812b" H 6350 4550 60  0000 C CNN
-F 2 "" H 6250 4850 60  0001 C CNN
+F 2 "symwaf:ws2812b" H 6250 4850 60  0001 C CNN
 F 3 "" H 6250 4850 60  0001 C CNN
 	1    6250 4850
@@
 $EndComp
 $Comp
-L ws2812b U?
+L ws2812b U12
 U 1 1 5AA40079
 P 7400 4850
-F 0 "U?" H 7200 5150 60  0000 C CNN
+F 0 "U12" H 7200 5150 60  0000 C CNN
 F 1 "ws2812b" H 7500 4550 60  0000 C CNN
-F 2 "" H 7400 4850 60  0001 C CNN
+F 2 "symwaf:ws2812b" H 7400 4850 60  0001 C CNN
 F 3 "" H 7400 4850 60  0001 C CNN
 	1    7400 4850
@@
 $EndComp
 $Comp
-L ws2812b U?
+L ws2812b U13
 U 1 1 5AA4007F
 P 8550 4850
-F 0 "U?" H 8350 5150 60  0000 C CNN
+F 0 "U13" H 8350 5150 60  0000 C CNN
 F 1 "ws2812b" H 8650 4550 60  0000 C CNN
-F 2 "" H 8550 4850 60  0001 C CNN
+F 2 "symwaf:ws2812b" H 8550 4850 60  0001 C CNN
 F 3 "" H 8550 4850 60  0001 C CNN
 	1    8550 4850
@@
 Connection ~ 2700 5400
 $Comp
-L C C?
+L C C13
 U 1 1 5AA411E6
 P 2900 4050
-F 0 "C?" H 2925 4150 50  0000 L CNN
+F 0 "C13" H 2925 4150 50  0000 L CNN
 F 1 "C" H 2925 3950 50  0000 L CNN
-F 2 "" H 2938 3900 50  0001 C CNN
+F 2 "Capacitors_SMD:C_0805" H 2938 3900 50  0001 C CNN
 F 3 "" H 2900 4050 50  0001 C CNN
 	1    2900 4050
@@
 	2900 4200 2900 4400
 $Comp
-L C C?
+L C C14
 U 1 1 5AA4141C
 P 4050 4050
-F 0 "C?" H 4075 4150 50  0000 L CNN
+F 0 "C14" H 4075 4150 50  0000 L CNN
 F 1 "C" H 4075 3950 50  0000 L CNN
-F 2 "" H 4088 3900 50  0001 C CNN
+F 2 "Capacitors_SMD:C_0805" H 4088 3900 50  0001 C CNN
 F 3 "" H 4050 4050 50  0001 C CNN
 	1    4050 4050
@@
 	4050 4200 4050 4400
 $Comp
-L C C?
+L C C15
 U 1 1 5AA414C9
 P 5200 4050
-F 0 "C?" H 5225 4150 50  0000 L CNN
+F 0 "C15" H 5225 4150 50  0000 L CNN
 F 1 "C" H 5225 3950 50  0000 L CNN
-F 2 "" H 5238 3900 50  0001 C CNN
+F 2 "Capacitors_SMD:C_0805" H 5238 3900 50  0001 C CNN
 F 3 "" H 5200 4050 50  0001 C CNN
 	1    5200 4050
@@
 	5200 4200 5200 4400
 $Comp
-L C C?
+L C C16
 U 1 1 5AA414D0
 P 6350 4050
-F 0 "C?" H 6375 4150 50  0000 L CNN
+F 0 "C16" H 6375 4150 50  0000 L CNN
 F 1 "C" H 6375 3950 50  0000 L CNN
-F 2 "" H 6388 3900 50  0001 C CNN
+F 2 "Capacitors_SMD:C_0805" H 6388 3900 50  0001 C CNN
 F 3 "" H 6350 4050 50  0001 C CNN
 	1    6350 4050
@@
 	6350 4200 6350 4400
 $Comp
-L C C?
+L C C17
 U 1 1 5AA416BF
 P 7500 4050
-F 0 "C?" H 7525 4150 50  0000 L CNN
+F 0 "C17" H 7525 4150 50  0000 L CNN
 F 1 "C" H 7525 3950 50  0000 L CNN
-F 2 "" H 7538 3900 50  0001 C CNN
+F 2 "Capacitors_SMD:C_0805" H 7538 3900 50  0001 C CNN
 F 3 "" H 7500 4050 50  0001 C CNN
 	1    7500 4050
@@
 	7500 4200 7500 4400
 $Comp
-L C C?
+L C C18
 U 1 1 5AA416C6
 P 8650 4050
-F 0 "C?" H 8675 4150 50  0000 L CNN
+F 0 "C18" H 8675 4150 50  0000 L CNN
 F 1 "C" H 8675 3950 50  0000 L CNN
-F 2 "" H 8688 3900 50  0001 C CNN
+F 2 "Capacitors_SMD:C_0805" H 8688 3900 50  0001 C CNN
 F 3 "" H 8650 4050 50  0001 C CNN
 	1    8650 4050
@@
 VCC
 $Comp
-L C C?
+L C C7
 U 1 1 5AA431E9
 P 2900 2150
-F 0 "C?" H 2925 2250 50  0000 L CNN
+F 0 "C7" H 2925 2250 50  0000 L CNN
 F 1 "C" H 2925 2050 50  0000 L CNN
-F 2 "" H 2938 2000 50  0001 C CNN
+F 2 "Capacitors_SMD:C_0805" H 2938 2000 50  0001 C CNN
 F 3 "" H 2900 2150 50  0001 C CNN
 	1    2900 2150
@@
 $EndComp
 $Comp
-L C C?
+L C C8
 U 1 1 5AA431F1
 P 4050 2150
-F 0 "C?" H 4075 2250 50  0000 L CNN
+F 0 "C8" H 4075 2250 50  0000 L CNN
 F 1 "C" H 4075 2050 50  0000 L CNN
-F 2 "" H 4088 2000 50  0001 C CNN
+F 2 "Capacitors_SMD:C_0805" H 4088 2000 50  0001 C CNN
 F 3 "" H 4050 2150 50  0001 C CNN
 	1    4050 2150
@@
 $EndComp
 $Comp
-L C C?
+L C C9
 U 1 1 5AA431F9
 P 5200 2150
-F 0 "C?" H 5225 2250 50  0000 L CNN
+F 0 "C9" H 5225 2250 50  0000 L CNN
 F 1 "C" H 5225 2050 50  0000 L CNN
-F 2 "" H 5238 2000 50  0001 C CNN
+F 2 "Capacitors_SMD:C_0805" H 5238 2000 50  0001 C CNN
 F 3 "" H 5200 2150 50  0001 C CNN
 	1    5200 2150
@@
 $EndComp
 $Comp
-L C C?
+L C C10
 U 1 1 5AA43201
 P 6350 2150
-F 0 "C?" H 6375 2250 50  0000 L CNN
+F 0 "C10" H 6375 2250 50  0000 L CNN
 F 1 "C" H 6375 2050 50  0000 L CNN
-F 2 "" H 6388 2000 50  0001 C CNN
+F 2 "Capacitors_SMD:C_0805" H 6388 2000 50  0001 C CNN
 F 3 "" H 6350 2150 50  0001 C CNN
 	1    6350 2150
@@
 $EndComp
 $Comp
-L C C?
+L C C11
 U 1 1 5AA43209
 P 7500 2150
-F 0 "C?" H 7525 2250 50  0000 L CNN
+F 0 "C11" H 7525 2250 50  0000 L CNN
 F 1 "C" H 7525 2050 50  0000 L CNN
-F 2 "" H 7538 2000 50  0001 C CNN
+F 2 "Capacitors_SMD:C_0805" H 7538 2000 50  0001 C CNN
 F 3 "" H 7500 2150 50  0001 C CNN
 	1    7500 2150
@@
 $EndComp
 $Comp
-L C C?
+L C C12
 U 1 1 5AA43211
 P 8650 2150
-F 0 "C?" H 8675 2250 50  0000 L CNN
+F 0 "C12" H 8675 2250 50  0000 L CNN
 F 1 "C" H 8675 2050 50  0000 L CNN
-F 2 "" H 8688 2000 50  0001 C CNN
+F 2 "Capacitors_SMD:C_0805" H 8688 2000 50  0001 C CNN
 F 3 "" H 8650 2150 50  0001 C CNN
 	1    8650 2150
